File: electronics/motor_driver_rpi_pi.sch (KiCad schematic (older format))
At the start: 18 parts, among them J5 Conn_02x20_Odd_Even, J6 Conn_02x20_Odd_Even, U1 DRV8833PWP

Commit message: update pcb file and netlist
Parts:
- C1, C4: footprint (none) -> Capacitor_SMD:C_1206_3216Metric
- C2, C3, C5, C6, C7: footprint (none) -> Capacitor_SMD:C_0805_2012Metric
- J5: footprint (none) -> Connector_PinSocket_2.54mm:PinSocket_2x20_P2.54mm_Vertical
- J6: footprint (none) -> Connector_PinHeader_2.54mm:PinHeader_2x20_P2.54mm_Vertical
Changed lines of the file:
@@
 F 0 "C5" V 7448 3200 50  0000 C CNN
 F 1 "2.2uF" V 7539 3200 50  0000 C CNN
-F 2 "" H 7738 3050 50  0001 C CNN
+F 2 "Capacitor_SMD:C_0805_2012Metric" H 7738 3050 50  0001 C CNN
 F 3 "~" H 7700 3200 50  0001 C CNN
 	1    7700 3200
@@
 F 0 "C4" V 6948 3200 50  0000 C CNN
 F 1 "10uF" V 7039 3200 50  0000 C CNN
-F 2 "" H 7238 3050 50  0001 C CNN
+F 2 "Capacitor_SMD:C_1206_3216Metric" H 7238 3050 50  0001 C CNN
 F 3 "~" H 7200 3200 50  0001 C CNN
 	1    7200 3200
@@
 F 0 "C7" V 9000 4900 50  0000 C CNN
 F 1 "100nF" V 9100 4900 50  0000 C CNN
-F 2 "" H 8888 4750 50  0001 C CNN
+F 2 "Capacitor_SMD:C_0805_2012Metric" H 8888 4750 50  0001 C CNN
 F 3 "~" H 8850 4900 50  0001 C CNN
 	1    8850 4900
@@
 F 0 "C6" V 8598 4100 50  0000 C CNN
 F 1 "100nF" V 8689 4100 50  0000 C CNN
-F 2 "" H 8888 3950 50  0001 C CNN
+F 2 "Capacitor_SMD:C_0805_2012Metric" H 8888 3950 50  0001 C CNN
 F 3 "~" H 8850 4100 50  0001 C CNN
 	1    8850 4100
@@
 F 0 "C3" H 7015 3546 50  0000 L CNN
 F 1 "10nF" H 7015 3455 50  0000 L CNN
-F 2 "" H 6938 3350 50  0001 C CNN
+F 2 "Capacitor_SMD:C_0805_2012Metric" H 6938 3350 50  0001 C CNN
 F 3 "~" H 6900 3500 50  0001 C CNN
 	1    6900 3500
@@
 F 0 "J5" H 3300 4167 50  0000 C CNN
 F 1 "Conn_02x20_Odd_Even" H 3300 4076 50  0000 C CNN
-F 2 "" H 3250 3050 50  0001 C CNN
+F 2 "Connector_PinSocket_2.54mm:PinSocket_2x20_P2.54mm_Vertical" H 3250 3050 50  0001 C CNN
 F 3 "~" H 3250 3050 50  0001 C CNN
 	1    3250 3050
@@
 F 0 "C1" V 4200 1600 50  0000 L CNN
 F 1 "10nF" V 4300 1600 50  0000 L CNN
-F 2 "" H 4488 1500 50  0001 C CNN
+F 2 "Capacitor_SMD:C_1206_3216Metric" H 4488 1500 50  0001 C CNN
 F 3 "~" H 4450 1650 50  0001 C CNN
 	1    4450 1650
@@
 F 0 "C2" V 4198 2150 50  0000 C CNN
 F 1 "100nF" V 4289 2150 50  0000 C CNN
-F 2 "" H 4488 2000 50  0001 C CNN
+F 2 "Capacitor_SMD:C_0805_2012Metric" H 4488 2000 50  0001 C CNN
 F 3 "~" H 4450 2150 50  0001 C CNN
 	1    4450 2150
@@
 F 0 "J6" H 3300 6667 50  0000 C CNN
 F 1 "Conn_02x20_Odd_Even" H 3300 6576 50  0000 C CNN
-F 2 "" H 3250 5550 50  0001 C CNN
+F 2 "Connector_PinHeader_2.54mm:PinHeader_2x20_P2.54mm_Vertical" H 3250 5550 50  0001 C CNN
 F 3 "~" H 3250 5550 50  0001 C CNN
 	1    3250 5550
